File: 250469-RevA/C64C-250469-01-A.sch (KiCad schematic (older format))
At the start: 0 parts

Commit message: Updates and BOMs
Changed lines of the file:
@@
 S 6650 4200 1150 800
 U 5E427C5E
-F0 "Video" 50
+F0 "Video - ClockGen" 50
 F1 "video.sch" 50
 $EndSheet
