File: 250469-RevA/cpu.sch (KiCad schematic (older format))
At the start: 6 parts, among them J6 Conn_02x22_Edge_Female, U3 74LS08, U6 8500

Commit message: Add initial PCB with placed components
Parts:
- J6: footprint 250469-01:Sullins_EBC22DRAS -> 250469-01:Sullins_EBC22DRAN
Changed lines of the file:
@@
 F 0 "J6" H 3250 4400 50  0000 C CNN
 F 1 "Conn_02x22_Edge_Female" H 3250 4250 50  0000 C CNN
-F 2 "250469-01:Sullins_EBC22DRAS" H 3200 3100 50  0001 C CNN
+F 2 "250469-01:Sullins_EBC22DRAN" H 3200 3100 50  0001 C CNN
 F 3 "~" H 3200 3100 50  0001 C CNN
 	1    3250 3100
