File: 250469-RevA/C64C-250469-01-A.kicad_pcb (KiCad board)
At the start: 2 copper layers, 390 x 135.9 mm, 134 parts, among them J1 Conn_01x20_Male, J10 LED, J2 Conn_02x12_Edge, J3 Conn_02x6_Edge, J4 DIN-6, J5 DIN-8, J6 Conn_02x22_Edge_Female, J7 DIN-7, J8 DB9_Female, J9 DB9_Female, M1 RF_Modulator, Q1 2SD313, Q2 2SC1815, Q3 2SC1815, Q5 2SC1384, U1 6526A, U10 41464, U11 41464, U18 4066, U19 2114, U2 6526A, U20 8701, U21 4066, U22 7416, U23 74LS14, U3 74LS08, U4 23128, U5 2332, U6 8500, U7 8565R2, U8 251715-01, U9 8580R5, Y1 Crystal

Commit message: More work on the PCB
Parts:
- added REF**: MountingHole_3.7mm_Pad, MountingHole:MountingHole_3.7mm_Pad, F.Cu at (188.6, 149.9)
- added REF**: MountingHole_3.7mm_Pad, MountingHole:MountingHole_3.7mm_Pad, F.Cu at (108.3, 149.8)
Other:
- board size 390 x 135.9 mm -> 390 x 134.9 mm
- board text added: "CIA1"
- board text added: "CIA2"
- board text added: "CPU"
- board text added: "Character ROM"
- board text added: "Color RAM"
- board text added: "KERNAL&BASIC"
- board text added: "Keyboard"
- board text added: "LED"
- board text added: "PLA"
- board text added: "RAM"
- board text added: "SID"
- board text added: "VIC2"
Changed lines of the file:
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@@
   (general
     (thickness 1.6)
-    (drawings 47)
+    (drawings 59)
     (tracks 0)
     (zones 0)
-    (modules 134)
+    (modules 136)
     (nets 206)
   )
@@
     (solder_mask_min_width 0.25)
     (aux_axis_origin 0 0)
-    (visible_elements FFFFFF7F)
+    (visible_elements FFFFF77F)
     (pcbplotparams
       (layerselection 0x010fc_ffffffff)
@@
     (add_net ~VIC)
   )
+  (module MountingHole:MountingHole_3.7mm_Pad (layer F.Cu)
+    (at 188.6 149.8583)
+    (descr "Mounting Hole 3.7mm")
+    (tags "mounting hole 3.7mm")
+    (attr virtual)
+    (fp_text reference REF** (at 0 -4.7) (layer F.SilkS)
+      (effects (font (size 1 1) (thickness 0.15)))
+    )
+    (fp_text value MountingHole_3.7mm_Pad (at 0 4.7) (layer F.Fab)
+      (effects (font (size 1 1) (thickness 0.15)))
+    )
+    (fp_circle (center 0 0) (end 3.95 0) (layer F.CrtYd) (width 0.05))
+    (fp_circle (center 0 0) (end 3.7 0) (layer Cmts.User) (width 0.15))
+    (fp_text user %R (at 0.3 0) (layer F.Fab)
+      (effects (font (size 1 1) (thickness 0.15)))
+    )
+    (pad 1 thru_hole circle (at 0 0) (size 7.4 7.4) (drill 3.7) (layers *.Cu *.Mask))
+  )
+  (module MountingHole:MountingHole_3.7mm_Pad (layer F.Cu)
+    (at 108.28 149.78)
+    (descr "Mounting Hole 3.7mm")
+    (tags "mounting hole 3.7mm")
+    (attr virtual)
+    (fp_text reference REF** (at 0 -4.7) (layer F.SilkS)
+      (effects (font (size 1 1) (thickness 0.15)))
+    )
+    (fp_text value MountingHole_3.7mm_Pad (at 0 4.7) (layer F.Fab)
+      (effects (font (size 1 1) (thickness 0.15)))
+    )
+    (fp_circle (center 0 0) (end 3.95 0) (layer F.CrtYd) (width 0.05))
+    (fp_circle (center 0 0) (end 3.7 0) (layer Cmts.User) (width 0.15))
+    (fp_text user %R (at 0.3 0) (layer F.Fab)
+      (effects (font (size 1 1) (thickness 0.15)))
+    )
+    (pad 1 thru_hole circle (at 0 0) (size 7.4 7.4) (drill 3.7) (layers *.Cu *.Mask))
+  )
   (module Symbol:KiCad-Logo_6mm_SilkScreen (layer F.Cu)
     (at 115.392514 167.3)
@@
     )
   )
+  (gr_text RAM (at 198.8 238.4 90) (layer F.SilkS)
+    (effects (font (size 1.1 1) (thickness 0.16)))
+  )
+  (gr_text Keyboard (at 404 229.975001 90) (layer F.SilkS)
+    (effects (font (size 1.1 1) (thickness 0.16)))
+  )
+  (gr_text LED (at 152.2 174.827) (layer F.SilkS)
+    (effects (font (size 1.1 1) (thickness 0.16)))
+  )
+  (gr_text KERNAL&BASIC (at 160.125 247.5) (layer F.SilkS)
+    (effects (font (size 1.1 1) (thickness 0.16)))
+  )
+  (gr_text "Character ROM" (at 138.6 247.6) (layer F.SilkS)
+    (effects (font (size 1.1 1) (thickness 0.16)))
+  )
+  (gr_text "Color RAM" (at 255.9 215.8) (layer F.SilkS)
+    (effects (font (size 1.1 1) (thickness 0.16)))
+  )
+  (gr_text CIA2 (at 115.225 247.5) (layer F.SilkS)
+    (effects (font (size 1.3 1.3) (thickness 0.18)))
+  )
+  (gr_text CPU (at 196.725 214.6) (layer F.SilkS)
+    (effects (font (size 1.3 1.3) (thickness 0.18)))
+  )
+  (gr_text PLA (at 234.125 254.8) (layer F.SilkS)
+    (effects (font (size 1.3 1.3) (thickness 0.18)))
+  )
+  (gr_text VIC2 (at 279.275 251.7) (layer F.SilkS)
+    (effects (font (size 1.3 1.3) (thickness 0.18)))
+  )
+  (gr_text SID (at 332.725 258.3) (layer F.SilkS)
+    (effects (font (size 1.3 1.3) (thickness 0.18)))
+  )
+  (gr_text CIA1 (at 368.925 258.4) (layer F.SilkS)
+    (effects (font (size 1.3 1.3) (thickness 0.18)))
+  )
   (gr_line (start 224.06616 129.6) (end 231.8 129.6) (layer Edge.Cuts) (width 0.1))
   (gr_line (start 222.65616 129.6) (end 222.90616 129.84988) (layer Edge.Cuts) (width 0.1))
@@
     (effects (font (size 2.7 2.5) (thickness 0.36)) (justify left))
   )
-  (gr_line (start 100 265.5) (end 490 265.5) (layer Edge.Cuts) (width 0.1))
+  (gr_line (start 100 264.5) (end 490 264.5) (layer Edge.Cuts) (width 0.1))
   (gr_line (start 120.5 141.5) (end 100 141.5) (layer Edge.Cuts) (width 0.1))
   (gr_line (start 120.5 141.5) (end 120.5 130.7) (layer Edge.Cuts) (width 0.1))
@@
   (gr_line (start 232.9 141.5) (end 232.9 130.7) (layer Edge.Cuts) (width 0.1))
   (gr_line (start 244.9 141.5) (end 232.9 141.5) (layer Edge.Cuts) (width 0.1))
-  (gr_line (start 100 141.5) (end 100 265.5) (layer Edge.Cuts) (width 0.1))
+  (gr_line (start 100 141.5) (end 100 264.5) (layer Edge.Cuts) (width 0.1))
   (gr_line (start 244.9 141.5) (end 244.9 129.6) (layer Edge.Cuts) (width 0.1))
   (gr_line (start 244.9 129.6) (end 382.4 129.6) (layer Edge.Cuts) (width 0.1))
@@
   (gr_line (start 453.5 158.7) (end 453.5 129.6) (layer Edge.Cuts) (width 0.1))
   (gr_line (start 453.5 129.6) (end 490 129.6) (layer Edge.Cuts) (width 0.1))
-  (gr_line (start 490 129.6) (end 490 265.5) (layer Edge.Cuts) (width 0.1))
+  (gr_line (start 490 129.6) (end 490 264.5) (layer Edge.Cuts) (width 0.1))
 )

Commit message: PCB: Add some more silkscreen labels
Other:
- board text added: "2114"
- board text added: "4066"
- board text added: "41464"
- board text added: "7416"
- board text added: "74LS08"
- board text added: "74LS14"
- board text added: "8701"
- board text added: "FUSE"
Changed lines of the file:
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@@
   (general
     (thickness 1.6)
-    (drawings 59)
+    (drawings 69)
     (tracks 0)
     (zones 0)
@@
     )
   )
+  (gr_text FUSE (at 449.4 195.4 90) (layer F.SilkS)
+    (effects (font (size 1.1 1) (thickness 0.16)))
+  )
+  (gr_text 74LS14 (at 143.2 191.2 90) (layer F.SilkS)
+    (effects (font (size 1.1 1) (thickness 0.16)))
+  )
+  (gr_text 74LS08 (at 217.4 170.4 90) (layer F.SilkS)
+    (effects (font (size 1.1 1) (thickness 0.16)))
+  )
+  (gr_text 7416 (at 239.4 171.6 90) (layer F.SilkS)
+    (effects (font (size 1.1 1) (thickness 0.16)))
+  )
+  (gr_text 4066 (at 256.5 171.5 90) (layer F.SilkS)
+    (effects (font (size 1.1 1) (thickness 0.16)))
+  )
+  (gr_text 4066 (at 386.4 212.4 90) (layer F.SilkS)
+    (effects (font (size 1.1 1) (thickness 0.16)))
+  )
+  (gr_text 8701 (at 299.2 235.5 90) (layer F.SilkS)
+    (effects (font (size 1.1 1) (thickness 0.16)))
+  )
+  (gr_text 2114 (at 255.9 230.5 90) (layer F.SilkS)
+    (effects (font (size 1.1 1) (thickness 0.16)))
+  )
+  (gr_text 41464 (at 206.6 238.1 90) (layer F.SilkS)
+    (effects (font (size 1.1 1) (thickness 0.16)))
+  )
+  (gr_text 41464 (at 190.8 238 90) (layer F.SilkS)
+    (effects (font (size 1.1 1) (thickness 0.16)))
+  )
   (gr_text RAM (at 198.8 238.4 90) (layer F.SilkS)

Commit message: Various improvements and changes to footprints
Parts:
- removed JP4: SolderJumper_2_Bridged, Jumper:SolderJumper-2_P1.3mm_Bridged_RoundedPad1.0x1.5mm
- CT1: footprint Capacitor_SMD:C_Trimmer_Voltronics_JZ -> krl_Capacitor_THT:C_Trimmer_JML_JML06_P5mm
- JP3: footprint Jumper:SolderJumper-2_P1.3mm_Bridged_RoundedPad1.0x1.5mm -> Connector_PinHeader_2.54mm:PinHeader_1x02_P2.54mm_Vertical
- moved CT1 3.36 mm to (315.2, 243.4)
- moved JP3 1.57 mm to (314.6, 251.3), turned to 270 degrees
- moved R17 0.30 mm to (149.3, 255.6)
Connections:
- U7 pad 19: Net-(JP4-Pad2) -> ~CAS

Commit message: Change footprint of PLA to Socket version
Parts:
- U8: footprint krl_Package_SPDIP:SPDIP-64_W19.05mm_LongPads -> krl_Package_SPDIP:SPDIP-64_W19.05mm_Socket_LongPads

Commit message: Corrected board dimensions and connector placements
The dimensions are now 100% correct after carefully measuring
a real board I acquired a few days ago.
Parts:
- added REF**: MountingHole_3.7mm, MountingHole:MountingHole_3.7mm, F.Cu at (475.2, 137.5)
- added REF**: MountingHole_3.7mm, MountingHole:MountingHole_3.7mm, F.Cu at (482.4, 137.8)
- moved J6 55.4 mm to (393.5, 108.3)
- moved J5 4.20 mm to (290.2, 142.1)
- moved J4 4.05 mm to (258.1, 142.1)
- moved M1 3.20 mm to (362.1, 162.4)
- moved C56 1.80 mm to (466.7, 137.5)
- moved J7 1.25 mm to (478.6, 150.6)
- moved J2 1.10 mm to (167.3, 135.3)
- moved CB1 1.08 mm to (473.0, 175.8)
- moved J3 1.01 mm to (229.2, 135.3)
- moved J8 0.55 mm to (478.6, 201.7)
- moved J9 0.45 mm to (478.6, 233.2)
Connections:
- CB1 pad : (no net) -> GND
- J7 pad 0: (no net) -> GND
Routing:
- net Net-(J7-Pad6): track 0.00 -> 9.27 mm
- net GND: vias 0 -> 5
- added copper zone on B.Cu, net GND
- added copper zone on F.Cu, net GND
- added copper zone on F.Cu, net Net-(C56-Pad1)
Other:
- board size 390 x 134.9 mm -> 390.6 x 136.2 mm

Commit message: Placed all mounting holes on the PCB
Parts:
- added REF**: MountingHole_3.5mm, MountingHole:MountingHole_3.5mm, F.Cu at (114.5, 261.2)
- added REF**: MountingHole_4mm, MountingHole:MountingHole_4mm, F.Cu at (105.2, 260.8)
- added REF**: MountingHole_3.5mm, MountingHole:MountingHole_3.5mm, F.Cu at (300.1, 260.7)
- added REF**: MountingHole_3.7mm, MountingHole:MountingHole_3.7mm, F.Cu at (485.7, 249.5)
- added REF**: MountingHole_4mm, MountingHole:MountingHole_4mm, F.Cu at (485.2, 260.6)
- added REF**: MountingHole_3.5mm, MountingHole:MountingHole_3.5mm, F.Cu at (281.1, 149.5)
- REF** (x2): value MountingHole_3.7mm_Pad -> MountingHole_3.5mm; footprint MountingHole:MountingHole_3.7mm_Pad -> MountingHole:MountingHole_3.5mm
- moved J6 56.0 mm to (391.1, 164.3)
- moved REF** 0.27 mm to (188.4, 149.7)
Other:
- outline, holes or cut-outs redrawn

Commit message: Right side routed
Parts:
- removed REF** (x5): MountingHole_3.5mm, MountingHole:MountingHole_3.5mm
- removed REF** (x3): MountingHole_3.7mm, MountingHole:MountingHole_3.7mm
- removed REF**: KiCad-Logo_6mm_SilkScreen, Symbol:KiCad-Logo_6mm_SilkScreen
- removed REF**: OSHW-Logo2_9.8x8mm_SilkScreen, Symbol:OSHW-Logo2_9.8x8mm_SilkScreen
- removed REF** (x2): MountingHole_4mm, MountingHole:MountingHole_4mm
- Q5: footprint Package_TO_SOT_THT:TO-92_Inline -> Package_TO_SOT_THT:TO-92_Inline_Wide
- moved C61 331.3 mm to (459.9, 197.5), turned to 270 degrees
- moved FL9 13.9 mm to (462.5, 240.4)
- moved FL8 13.3 mm to (462.5, 244.9)
- moved FL1 13.2 mm to (462.5, 226.9)
- moved FL7 12.8 mm to (462.5, 249.4)
- moved FL6 12.1 mm to (462.5, 253.8)
- moved FL4 11.5 mm to (462.5, 210.2)
- moved FL3 11.0 mm to (462.5, 214.7)
- moved D2 11.0 mm to (441.2, 198.3), turned to 180 degrees
- moved FL2 10.5 mm to (462.5, 219.2)
- moved FL5 9.96 mm to (462.5, 231.4)
- moved RN4 9.84 mm to (397.1, 175.4)
- moved D4 8.50 mm to (431.6, 206.5)
- moved C63 6.32 mm to (438.5, 221.5)
- moved D7 6.14 mm to (425.2, 222.7)
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Connections:
- CB1 pad : GND -> (no net)
- CB1 pad 2: 9V_AC1 -> +5V
- CB1 pad 5: +5V -> 9V_AC1
- J7 pad 0: GND -> (no net)
- L1 pad 6: Net-(CB1-Pad4) -> Net-(CB1-Pad3)
- L1 pad 7: Net-(CB1-Pad1) -> Net-(CB1-Pad6)
- Q1 pad 1: /Tape - Serial/MOTOR -> Net-(D1-Pad1)
- Q1 pad 3: Net-(D1-Pad1) -> /Tape - Serial/MOTOR
- Q5 pad 1: Net-(C66-Pad1) -> +9V
- Q5 pad 2: Net-(D7-Pad1) -> Net-(C66-Pad1)
- Q5 pad 3: +9V -> Net-(D7-Pad1)
- R19 pad 1: Net-(CB1-Pad6) -> Net-(CB1-Pad1)
Routing:
- net +5V: track 0.00 -> 195.2 mm, vias 0 -> 1
- net ROW4: track 0.00 -> 166.6 mm, vias 0 -> 1
- net ROW1: track 0.00 -> 148.1 mm, vias 0 -> 1
- net ROW2: track 0.00 -> 144.4 mm, vias 0 -> 1
- net /Joystick Ports/POT_AY: track 0.00 -> 142.0 mm, vias 0 -> 1
- net /Joystick Ports/POT_AX: track 0.00 -> 138.4 mm, vias 0 -> 1
- net ROW0: track 0.00 -> 137.6 mm, vias 0 -> 1
- net ROW3: track 0.00 -> 133.4 mm, vias 0 -> 2
- net COL2: track 0.00 -> 129.3 mm, vias 0 -> 1
- net COL3: track 0.00 -> 129.1 mm, vias 0 -> 1
- net COL1: track 0.00 -> 126.4 mm, vias 0 -> 1
- net /Joystick Ports/POT_BX: track 0.00 -> 118.0 mm
- net D7: track 0.00 -> 117.4 mm
- net D6: track 0.00 -> 115.4 mm
- net D5: track 0.00 -> 113.5 mm
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- added copper zone on B.Cu, net +5V
- removed copper zone on B.Cu, net GND
- removed copper zone on F.Cu, net GND
- removed copper zone on F.Cu, net Net-(C56-Pad1)
Other:
- board text added: "E C B"
