File: 250469-RevA/tape_serial.sch (KiCad schematic (older format))
At the start: 21 parts, among them J3 Conn_02x6_Edge, J4 DIN-6, Q1 2SD313, Q2 2SC1815

Commit message: Changed footprint of DIC connectors and wiring of Color RAM
Parts:
- J4: footprint krl_Connector_DIN:CUI-Devices_SDS-60J_DIN-6_Circular -> krl_Connector_DIN:C64_Original_DIN-6_Circular
Changed lines of the file:
@@
 F 0 "J4" H 5350 2900 50  0000 C CNN
 F 1 "DIN-6" H 5750 2400 50  0000 C CNN
-F 2 "krl_Connector_DIN:CUI-Devices_SDS-60J_DIN-6_Circular" H 5500 2650 50  0001 C CNN
+F 2 "krl_Connector_DIN:C64_Original_DIN-6_Circular" H 5500 2650 50  0001 C CNN
 F 3 "http://www.mouser.com/ds/2/18/40_c091_abd_e-75918.pdf" H 5500 2650 50  0001 C CNN
 	1    5500 2650
