File: 250469-RevA/audio.sch (KiCad schematic (older format))
At the start: 16 parts, among them Q3 2SC1815, U9 8580R5

Commit message: Updates and BOMs
Parts:
- C77: footprint Capacitor_THT:CP_Radial_D8.0mm_P5.00mm -> Capacitor_THT:CP_Radial_D10.0mm_P5.00mm
Changed lines of the file:
@@
 F 0 "C77" V 8255 4575 50  0000 C CNN
 F 1 "10u" V 8164 4575 50  0000 C CNN
-F 2 "Capacitor_THT:CP_Radial_D8.0mm_P5.00mm" H 8038 4425 50  0001 C CNN
+F 2 "Capacitor_THT:CP_Radial_D10.0mm_P5.00mm" H 8038 4425 50  0001 C CNN
 F 3 "~" H 8000 4575 50  0001 C CNN
 	1    8000 4575

Commit message: Update schematic after changes in libs
Parts:
- C77: symbol Device:CP -> Device:C_Polarized
Changed lines of the file:
@@
 $EndComp
 $Comp
-L Device:CP C77
+L Device:C_Polarized C77
 U 1 1 5E57628A
 P 8000 4575
+AR Path="/5E57628A" Ref="C77"  Part="1"
+AR Path="/5E6244E0/5E57628A" Ref="C77"  Part="1"
 F 0 "C77" V 8255 4575 50  0000 C CNN
 F 1 "10u" V 8164 4575 50  0000 C CNN
