File: 250469-RevA/joystick.sch (KiCad schematic (older format))
At the start: 17 parts, among them J8 DB9_Female, J9 DB9_Female, U18 4066

Commit message: Updates and BOMs
Parts:
- L3: value Choke Coil -> 10uH; footprint Inductor_THT:L_Axial_L9.5mm_D4.0mm_P12.70mm_Horizontal_Fastron_SMCC -> 250469-01:L_Radial_L7.5mm_W3mm_P5.00mm_Kemet_SBT-02
Changed lines of the file:
@@
 AR Path="/5E6B96A5/5E6DF147" Ref="L3"  Part="1"
 F 0 "L3" V 9550 5800 50  0000 C CNN
-F 1 "Choke Coil" V 9350 5800 50  0000 C CNN
-F 2 "Inductor_THT:L_Axial_L9.5mm_D4.0mm_P12.70mm_Horizontal_Fastron_SMCC" H 9450 5800 50  0001 C CNN
+F 1 "10uH" V 9350 5800 50  0000 C CNN
+F 2 "250469-01:L_Radial_L7.5mm_W3mm_P5.00mm_Kemet_SBT-02" H 9450 5800 50  0001 C CNN
 F 3 "~" H 9450 5800 50  0001 C CNN
 	1    9450 5800

Commit message: Update schematic after changes in libs
Parts:
- FL1, FL2, FL3, FL4, FL5, FL6, FL7, FL8, FL9: symbol Device:EMI_Filter_LCL -> Device:Filter_EMI_LCL
Changed lines of the file:
@@
 $EndComp
 $Comp
-L Device:EMI_Filter_LCL FL?
+L Device:Filter_EMI_LCL FL?
 U 1 1 5E6DF074
 P 3800 2350
 AR Path="/5E1CEE0C/5E6DF074" Ref="FL?"  Part="1"
 AR Path="/5E6B96A5/5E6DF074" Ref="FL4"  Part="1"
+AR Path="/5E6DF074" Ref="FL4"  Part="1"
 F 0 "FL4" H 3550 2300 50  0000 C CNN
 F 1 "270p" H 3800 2576 50  0000 C CNN
@@
 $EndComp
 $Comp
-L Device:EMI_Filter_LCL FL?
+L Device:Filter_EMI_LCL FL?
 U 1 1 5E6DF07A
 P 3800 3100
 AR Path="/5E1CEE0C/5E6DF07A" Ref="FL?"  Part="1"
 AR Path="/5E6B96A5/5E6DF07A" Ref="FL3"  Part="1"
+AR Path="/5E6DF07A" Ref="FL3"  Part="1"
 F 0 "FL3" H 3550 3050 50  0000 C CNN
 F 1 "270p" H 3800 3326 50  0000 C CNN
@@
 $EndComp
 $Comp
-L Device:EMI_Filter_LCL FL?
+L Device:Filter_EMI_LCL FL?
 U 1 1 5E6DF080
 P 3800 4250
 AR Path="/5E1CEE0C/5E6DF080" Ref="FL?"  Part="1"
 AR Path="/5E6B96A5/5E6DF080" Ref="FL5"  Part="1"
+AR Path="/5E6DF080" Ref="FL5"  Part="1"
 F 0 "FL5" H 3550 4200 50  0000 C CNN
 F 1 "270p" H 3800 4476 50  0000 C CNN
@@
 $EndComp
 $Comp
-L Device:EMI_Filter_LCL FL?
+L Device:Filter_EMI_LCL FL?
 U 1 1 5E6DF086
 P 4550 4850
 AR Path="/5E1CEE0C/5E6DF086" Ref="FL?"  Part="1"
 AR Path="/5E6B96A5/5E6DF086" Ref="FL1"  Part="1"
+AR Path="/5E6DF086" Ref="FL1"  Part="1"
 F 0 "FL1" H 4300 4800 50  0000 C CNN
 F 1 "270p" H 4550 5076 50  0000 C CNN
@@
 $EndComp
 $Comp
-L Device:EMI_Filter_LCL FL?
+L Device:Filter_EMI_LCL FL?
 U 1 1 5E6DF08C
 P 4550 3650
 AR Path="/5E1CEE0C/5E6DF08C" Ref="FL?"  Part="1"
 AR Path="/5E6B96A5/5E6DF08C" Ref="FL2"  Part="1"
+AR Path="/5E6DF08C" Ref="FL2"  Part="1"
 F 0 "FL2" H 4300 3600 50  0000 C CNN
 F 1 "270p" H 4550 3876 50  0000 C CNN
@@
 (CONTROL PORT 1)
 $Comp
-L Device:EMI_Filter_LCL FL?
+L Device:Filter_EMI_LCL FL?
 U 1 1 5E6DF122
 P 8400 5550
 AR Path="/5E1CEE0C/5E6DF122" Ref="FL?"  Part="1"
 AR Path="/5E6B96A5/5E6DF122" Ref="FL6"  Part="1"
+AR Path="/5E6DF122" Ref="FL6"  Part="1"
 F 0 "FL6" H 8150 5500 50  0000 C CNN
 F 1 "270p" H 8400 5776 50  0000 C CNN
@@
 $EndComp
 $Comp
-L Device:EMI_Filter_LCL FL?
+L Device:Filter_EMI_LCL FL?
 U 1 1 5E6DF12E
 P 9050 4650
 AR Path="/5E1CEE0C/5E6DF12E" Ref="FL?"  Part="1"
 AR Path="/5E6B96A5/5E6DF12E" Ref="FL7"  Part="1"
+AR Path="/5E6DF12E" Ref="FL7"  Part="1"
 F 0 "FL7" H 8800 4600 50  0000 C CNN
 F 1 "270p" H 9050 4876 50  0000 C CNN
@@
 $EndComp
 $Comp
-L Device:EMI_Filter_LCL FL?
+L Device:Filter_EMI_LCL FL?
 U 1 1 5E6DF134
 P 8600 3950
 AR Path="/5E1CEE0C/5E6DF134" Ref="FL?"  Part="1"
 AR Path="/5E6B96A5/5E6DF134" Ref="FL8"  Part="1"
+AR Path="/5E6DF134" Ref="FL8"  Part="1"
 F 0 "FL8" H 8350 3900 50  0000 C CNN
 F 1 "270p" H 8600 4176 50  0000 C CNN
@@
 $EndComp
 $Comp
-L Device:EMI_Filter_LCL FL?
+L Device:Filter_EMI_LCL FL?
 U 1 1 5E6DF17C
 P 9100 3350
 AR Path="/5E1CEE0C/5E6DF17C" Ref="FL?"  Part="1"
 AR Path="/5E6B96A5/5E6DF17C" Ref="FL9"  Part="1"
+AR Path="/5E6DF17C" Ref="FL9"  Part="1"
 F 0 "FL9" H 8850 3300 50  0000 C CNN
 F 1 "270p" H 9100 3576 50  0000 C CNN
