File: 250469-RevA/keyboard.sch (KiCad schematic (older format))
At the start: 9 parts, among them J1 Conn_01x20_Male, U1 6526A, U23 74LS14

Commit message: Updates and BOMs
Parts:
- removed D6: Vz=3V, Diode_THT:D_DO-35_SOD27_P5.08mm_Vertical_KathodeUp, symbol Device:D_Zener
- added D6: RD3.0EB1, Diode_THT:D_DO-35_SOD27_P5.08mm_Vertical_KathodeUp, symbol krl_Diode:RD3.0EB1
- L4: value Choke Coil -> 10uH; footprint Inductor_THT:L_Axial_L9.5mm_D4.0mm_P12.70mm_Horizontal_Fastron_SMCC -> 250469-01:L_Radial_L7.5mm_W3mm_P5.00mm_Kemet_SBT-02
- U1: footprint Package_DIP:DIP-40_W15.24mm -> Package_DIP:DIP-40_W15.24mm_Socket
Other:
- moved on the sheet: C44, R16, U23A
Changed lines of the file:
@@
 AR Path="/5E4C440A/5E4CF21E" Ref="L4"  Part="1"
 F 0 "L4" V 2900 6450 50  0000 C CNN
-F 1 "Choke Coil" V 2700 6450 50  0000 C CNN
-F 2 "Inductor_THT:L_Axial_L9.5mm_D4.0mm_P12.70mm_Horizontal_Fastron_SMCC" H 2800 6450 50  0001 C CNN
+F 1 "10uH" V 2700 6450 50  0000 C CNN
+F 2 "250469-01:L_Radial_L7.5mm_W3mm_P5.00mm_Kemet_SBT-02" H 2800 6450 50  0001 C CNN
 F 3 "~" H 2800 6450 50  0001 C CNN
 	1    2800 6450
@@
 L 74xx:74LS14 U23
 U 1 1 5E4D932C
-P 6450 4000
-F 0 "U23" H 6450 4317 50  0000 C CNN
-F 1 "74LS14" H 6450 4226 50  0000 C CNN
-F 2 "Package_DIP:DIP-14_W7.62mm_Socket" H 6450 4000 50  0001 C CNN
-F 3 "http://www.ti.com/lit/gpn/sn74LS14" H 6450 4000 50  0001 C CNN
-	1    6450 4000
+P 6500 4000
+F 0 "U23" H 6500 4317 50  0000 C CNN
+F 1 "74LS14" H 6500 4226 50  0000 C CNN
+F 2 "Package_DIP:DIP-14_W7.62mm_Socket" H 6500 4000 50  0001 C CNN
+F 3 "http://www.ti.com/lit/gpn/sn74LS14" H 6500 4000 50  0001 C CNN
+	1    6500 4000
 	1    0    0    -1
 $EndComp
@@
 L Device:CP C44
 U 1 1 5E4D9333
-P 5950 4200
-F 0 "C44" H 6068 4246 50  0000 L CNN
-F 1 "2.2u" H 6068 4155 50  0000 L CNN
-F 2 "Capacitor_THT:CP_Radial_D8.0mm_P5.00mm" H 5988 4050 50  0001 C CNN
-F 3 "~" H 5950 4200 50  0001 C CNN
-	1    5950 4200
-	1    0    0    -1
-$EndComp
-$Comp
-L Device:D_Zener D6
-U 1 1 5E4D9339
-P 5550 4350
-F 0 "D6" V 5504 4430 50  0000 L CNN
-F 1 "Vz=3V" V 5595 4430 50  0000 L CNN
-F 2 "Diode_THT:D_DO-35_SOD27_P5.08mm_Vertical_KathodeUp" H 5550 4350 50  0001 C CNN
-F 3 "~" H 5550 4350 50  0001 C CNN
-	1    5550 4350
-	0    1    1    0
+P 5950 4350
+F 0 "C44" H 6068 4396 50  0000 L CNN
+F 1 "2.2u" H 6068 4305 50  0000 L CNN
+F 2 "Capacitor_THT:CP_Radial_D8.0mm_P5.00mm" H 5988 4200 50  0001 C CNN
+F 3 "~" H 5950 4350 50  0001 C CNN
+	1    5950 4350
+	1    0    0    -1
 $EndComp
 $Comp
@@
 L power:GND #PWR0115
 U 1 1 5E4D9345
-P 5950 4650
-F 0 "#PWR0115" H 5950 4400 50  0001 C CNN
-F 1 "GND" H 5955 4477 50  0000 C CNN
-F 2 "" H 5950 4650 50  0001 C CNN
-F 3 "" H 5950 4650 50  0001 C CNN
-	1    5950 4650
+P 5950 4700
+F 0 "#PWR0115" H 5950 4450 50  0001 C CNN
+F 1 "GND" H 5955 4527 50  0000 C CNN
+F 2 "" H 5950 4700 50  0001 C CNN
+F 3 "" H 5950 4700 50  0001 C CNN
+	1    5950 4700
 	1    0    0    -1
 $EndComp
@@
 L Device:R R16
 U 1 1 5E4D934C
-P 5250 4000
-F 0 "R16" V 5043 4000 50  0000 C CNN
-F 1 "560" V 5134 4000 50  0000 C CNN
-F 2 "Resistor_THT:R_Axial_DIN0207_L6.3mm_D2.5mm_P5.08mm_Vertical" V 5180 4000 50  0001 C CNN
-F 3 "~" H 5250 4000 50  0001 C CNN
-	1    5250 4000
+P 5050 4000
+F 0 "R16" V 4843 4000 50  0000 C CNN
+F 1 "560" V 4934 4000 50  0000 C CNN
+F 2 "Resistor_THT:R_Axial_DIN0207_L6.3mm_D2.5mm_P5.08mm_Vertical" V 4980 4000 50  0001 C CNN
+F 3 "~" H 5050 4000 50  0001 C CNN
+	1    5050 4000
 	0    1    1    0
 $EndComp
 Wire Wire Line
-	5400 4000 5550 4000
-Wire Wire Line
-	5950 4050 5950 4000
+	5200 4000 5500 4000
+Wire Wire Line
+	5950 4200 5950 4000
 Connection ~ 5950 4000
 Wire Wire Line
-	5950 4000 6150 4000
-Wire Wire Line
-	5550 4200 5550 4000
-Connection ~ 5550 4000
-Wire Wire Line
-	5550 4000 5950 4000
-Wire Wire Line
-	5950 4350 5950 4550
-Wire Wire Line
-	5550 4500 5550 4550
-Wire Wire Line
-	5550 4550 5950 4550
-Connection ~ 5950 4550
-Wire Wire Line
-	5950 4550 5950 4650
+	5950 4000 6200 4000
+Wire Wire Line
+	5500 4200 5500 4000
+Connection ~ 5500 4000
+Wire Wire Line
+	5500 4000 5950 4000
+Wire Wire Line
+	5950 4500 5950 4600
+Wire Wire Line
+	5500 4500 5500 4600
+Wire Wire Line
+	5500 4600 5950 4600
+Connection ~ 5950 4600
+Wire Wire Line
+	5950 4600 5950 4700
 Wire Bus Line
 	6750 2000 7250 2000
@@
 ~SRQ
 Wire Wire Line
-	6750 4000 7300 4000
+	6800 4000 7300 4000
 Wire Wire Line
 	7650 5050 6950 5050
@@
 	4600 4000 4600 3950
 Wire Wire Line
-	4600 4000 5100 4000
+	4600 4000 4900 4000
 $Comp
 L krl_MOS-Technology:6526A U1
@@
 F 0 "U1" H 8050 4250 50  0000 C CNN
 F 1 "6526A" H 8700 4250 50  0000 C CNN
-F 2 "Package_DIP:DIP-40_W15.24mm" H 7600 1900 50  0001 C CIN
+F 2 "Package_DIP:DIP-40_W15.24mm_Socket" H 7600 1900 50  0001 C CIN
 F 3 "http://www.6502.org/documents/datasheets/mos/mos_6526_cia.pdf" H 8350 3700 50  0001 C CNN
 F 4 "906108" H 8400 3100 50  0001 C CNN "ProductCodes"
@@
 Wire Wire Line
 	7650 4100 7900 4100
+$Comp
+L krl_Diode:RD3.0EB1 D6
+U 1 1 5EA1E54E
+P 5500 4350
+F 0 "D6" V 5450 4150 50  0000 L CNN
+F 1 "RD3.0EB1" V 5550 3900 50  0000 L CNN
+F 2 "Diode_THT:D_DO-35_SOD27_P5.08mm_Vertical_KathodeUp" H 5500 4125 50  0001 C CIN
+F 3 "" H 5500 4350 50  0001 C CNN
+F 4 "1N5225B" H 5500 4550 50  0001 C CNN "Equivalent"
+	1    5500 4350
+	0    1    1    0
+$EndComp
 Wire Bus Line
 	9200 2850 9200 3200

Commit message: Update schematic after changes in libs
Parts:
- C44, C59: symbol Device:CP -> Device:C_Polarized
Changed lines of the file:
@@
 $EndComp
 $Comp
-L Device:CP C?
+L Device:C_Polarized C?
 U 1 1 5E4CF224
 P 3850 6700
 AR Path="/5E1CEE0C/5E4CF224" Ref="C?"  Part="1"
 AR Path="/5E4C440A/5E4CF224" Ref="C59"  Part="1"
+AR Path="/5E4CF224" Ref="C59"  Part="1"
 F 0 "C59" H 3968 6746 50  0000 L CNN
 F 1 "4.7u" H 3968 6655 50  0000 L CNN
@@
 $EndComp
 $Comp
-L Device:CP C44
+L Device:C_Polarized C44
 U 1 1 5E4D9333
 P 5950 4350
+AR Path="/5E4D9333" Ref="C44"  Part="1"
+AR Path="/5E4C440A/5E4D9333" Ref="C44"  Part="1"
 F 0 "C44" H 6068 4396 50  0000 L CNN
 F 1 "2.2u" H 6068 4305 50  0000 L CNN
