File: 250469-RevA/power.sch (KiCad schematic (older format))
At the start: 24 parts, among them J10 LED, J7 DIN-7, Q5 2SC1384, U18 4066, U21 4066, U22 7416, U23 74LS14, U3 74LS08

Commit message: Updates and BOMs
Parts:
- removed D2: GBL06-E3/45, Diode_THT:Diode_Bridge_Vishay_GBL, symbol krl_Diode_Bridge:GBL06
- added D2: 2W02G-E4/51, Diode_THT:Diode_Bridge_Round_D9.8mm, symbol Device:D_Bridge_+A-A
- C65: footprint Capacitor_THT:CP_Radial_D12.5mm_P7.50mm -> Capacitor_THT:CP_Radial_D10.0mm_P5.00mm
- C66: footprint Capacitor_THT:CP_Radial_D12.5mm_P7.50mm -> Capacitor_THT:CP_Radial_D12.5mm_P5.00mm
- D3, D4: footprint Diode_THT:D_DO-35_SOD27_P5.08mm_Vertical_KathodeUp -> Diode_THT:D_DO-41_SOD81_P5.08mm_Vertical_KathodeUp
- D7: footprint Diode_THT:D_DO-35_SOD27_P5.08mm_Vertical_KathodeUp -> Diode_THT:D_DO-34_SOD68_P5.08mm_Vertical_KathodeUp
Changed lines of the file:
@@
 F 0 "C65" V 5945 1800 50  0000 C CNN
 F 1 "220u" V 6036 1800 50  0000 C CNN
-F 2 "Capacitor_THT:CP_Radial_D12.5mm_P7.50mm" H 6238 1650 50  0001 C CNN
+F 2 "Capacitor_THT:CP_Radial_D10.0mm_P5.00mm" H 6238 1650 50  0001 C CNN
 F 3 "~" H 6200 1800 50  0001 C CNN
 	1    6200 1800
@@
 F 0 "D3" H 7200 2017 50  0000 C CNN
 F 1 "1N4001" H 7200 1926 50  0000 C CNN
-F 2 "Diode_THT:D_DO-35_SOD27_P5.08mm_Vertical_KathodeUp" H 7200 1625 50  0001 C CNN
+F 2 "Diode_THT:D_DO-41_SOD81_P5.08mm_Vertical_KathodeUp" H 7200 1625 50  0001 C CNN
 F 3 "http://www.vishay.com/docs/88503/1n4001.pdf" H 7200 1800 50  0001 C CNN
 	1    7200 1800
@@
 F 0 "D4" V 6604 2130 50  0000 L CNN
 F 1 "1N4001" V 6695 2130 50  0000 L CNN
-F 2 "Diode_THT:D_DO-35_SOD27_P5.08mm_Vertical_KathodeUp" H 6650 1875 50  0001 C CNN
+F 2 "Diode_THT:D_DO-41_SOD81_P5.08mm_Vertical_KathodeUp" H 6650 1875 50  0001 C CNN
 F 3 "http://www.vishay.com/docs/88503/1n4001.pdf" H 6650 2050 50  0001 C CNN
 	1    6650 2050
@@
 F 0 "C66" H 8068 1496 50  0000 L CNN
 F 1 "330u/35V" H 8068 1405 50  0000 L CNN
-F 2 "Capacitor_THT:CP_Radial_D12.5mm_P7.50mm" H 7988 1300 50  0001 C CNN
+F 2 "Capacitor_THT:CP_Radial_D12.5mm_P5.00mm" H 7988 1300 50  0001 C CNN
 F 3 "~" H 7950 1450 50  0001 C CNN
 	1    7950 1450
@@
 F 0 "D7" V 9250 1710 50  0000 L CNN
 F 1 "RD10ESB2" V 9340 1420 50  0000 L CNN
-F 2 "Diode_THT:D_DO-35_SOD27_P5.08mm_Vertical_KathodeUp" H 9300 1725 50  0001 C CNN
+F 2 "Diode_THT:D_DO-34_SOD68_P5.08mm_Vertical_KathodeUp" H 9300 1725 50  0001 C CNN
 F 3 "" H 9300 1900 50  0001 C CNN
 	1    9300 1900
@@
 Used to\ndischarge C58
 $Comp
-L krl_Diode_Bridge:GBL06 D2
-U 1 1 5E9A6E0C
+L Device:D_Bridge_+A-A D2
+U 1 1 5E9E6D2E
 P 5650 2300
-F 0 "D2" H 5825 2550 50  0000 L CNN
-F 1 "GBL06-E3/45" H 5825 2475 50  0000 L CNN
-F 2 "Diode_THT:Diode_Bridge_Vishay_GBL" H 5800 2425 50  0001 L CNN
-F 3 "http://www.vishay.com/docs/88609/gbl005.pdf" H 5650 2300 50  0001 C CNN
+F 0 "D2" H 5994 2346 50  0000 L CNN
+F 1 "2W02G-E4/51" H 5994 2255 50  0000 L CNN
+F 2 "Diode_THT:Diode_Bridge_Round_D9.8mm" H 5650 2300 50  0001 C CNN
+F 3 "~" H 5650 2300 50  0001 C CNN
 	1    5650 2300
 	1    0    0    -1

Commit message: Add initial PCB with placed components
Parts:
- Q5: footprint Package_TO_SOT_THT:TO-92 -> Package_TO_SOT_THT:TO-92_Inline
Changed lines of the file:
@@
 F 0 "Q5" V 9629 1300 50  0000 C CNN
 F 1 "2SC1384" V 9538 1300 50  0000 C CNN
-F 2 "Package_TO_SOT_THT:TO-92" H 9500 1225 50  0001 L CIN
+F 2 "Package_TO_SOT_THT:TO-92_Inline" H 9500 1225 50  0001 L CIN
 F 3 "http://www.unisonic.com.tw/datasheet/2SC1384.pdf" H 9300 1300 50  0001 L CNN
 	1    9300 1300

Commit message: Change label in Power section
Other:
- note added: "POWER"
- note removed: "Power"
Changed lines of the file:
@@
 	9100 5200 9100 5600
 Text Notes 1250 1250 0    200  ~ 0
-Power
+POWER
 Text Notes 8400 4400 0    100  ~ 0
 LED Connector

Commit message: Changes after updates in the KRL
Connections:
- net +5V: now also CB1.2 (B); no longer CB1.5 (B)
- net 9V_AC1: now also CB1.5 (B); no longer CB1.2 (B)
- net at L1.6: now also CB1.3 (C); no longer CB1.4 (A)
- net at L1.7: now also CB1.6 (C); no longer CB1.1 (A)
- net at R19.1: now also CB1.1 (A); no longer CB1.6 (C)
Changed lines of the file:
@@
 	1    0    0    -1
-$EndComp
-$Comp
-L krl_Switch:SW_DPDT CB1
-U 1 1 5E630F46
-P 4250 3350
-F 0 "CB1" H 4250 3750 50  0000 C CNN
-F 1 "SW_DPDT" V 3876 3350 50  0001 C CNN
-F 2 "250469-01:RockerSwitch_CuK_DPDT_E201J1AV2" H 4550 3250 50  0001 C CNN
-F 3 "~" H 4500 3350 50  0001 C CNN
-	1    4250 3350
-	-1   0    0    -1
 $EndComp
 Wire Wire Line
@@
 U 1 1 5E795972
 P 9300 1300
+AR Path="/5E795972" Ref="Q5"  Part="1"
+AR Path="/5E8458FD/5E795972" Ref="Q5"  Part="1"
 F 0 "Q5" V 9629 1300 50  0000 C CNN
 F 1 "2SC1384" V 9538 1300 50  0000 C CNN
@@
 	1    0    0    -1
 $EndComp
+$Comp
+L krl_Switch:SW_DPDT CB1
+U 1 1 5EC8C9AB
+P 4250 3350
+F 0 "CB1" H 4250 3750 50  0000 C CNN
+F 1 "SW_DPDT" V 3876 3350 50  0001 C CNN
+F 2 "250469-01:RockerSwitch_CuK_DPDT_E201J1AV2" H 4550 3250 50  0001 C CNN
+F 3 "~" H 4500 3350 50  0001 C CNN
+	1    4250 3350
+	-1   0    0    1
+$EndComp
 $EndSCHEMATC

Commit message: Right side routed
Parts:
- Q5: footprint Package_TO_SOT_THT:TO-92_Inline -> Package_TO_SOT_THT:TO-92_Inline_Wide
Changed lines of the file:
@@
 F 0 "Q5" V 9629 1300 50  0000 C CNN
 F 1 "2SC1384" V 9538 1300 50  0000 C CNN
-F 2 "Package_TO_SOT_THT:TO-92_Inline" H 9500 1225 50  0001 L CIN
+F 2 "Package_TO_SOT_THT:TO-92_Inline_Wide" H 9500 1225 50  0001 L CIN
 F 3 "http://www.unisonic.com.tw/datasheet/2SC1384.pdf" H 9300 1300 50  0001 L CNN
 	1    9300 1300

Commit message: Changed footprint of DIC connectors and wiring of Color RAM
Parts:
- J7: footprint krl_Connector_DIN:CUI-Devices_SDS-70J_DIN-7_Circular -> krl_Connector_DIN:C64_Original_DIN-7_Circular
Changed lines of the file:
@@
 F 0 "J7" H 1650 2583 50  0000 C CNN
 F 1 "DIN-7" H 1650 2674 50  0000 C CNN
-F 2 "krl_Connector_DIN:CUI-Devices_SDS-70J_DIN-7_Circular" H 1650 2950 50  0001 C CNN
+F 2 "krl_Connector_DIN:C64_Original_DIN-7_Circular" H 1650 2950 50  0001 C CNN
 F 3 "http://www.mouser.com/ds/2/18/40_c091_abd_e-75918.pdf" H 1650 2950 50  0001 C CNN
 	1    1650 2950

Commit message: Update schematic after changes in libs
Parts:
- C58, C63, C65, C66: symbol Device:CP -> Device:C_Polarized
Changed lines of the file:
@@
 $EndComp
 $Comp
-L Device:CP C58
+L Device:C_Polarized C58
 U 1 1 5E62570C
 P 4600 4300
+AR Path="/5E62570C" Ref="C58"  Part="1"
+AR Path="/5E8458FD/5E62570C" Ref="C58"  Part="1"
 F 0 "C58" H 4718 4346 50  0000 L CNN
 F 1 "100u/16V" H 4718 4255 50  0000 L CNN
@@
 	5650 1000 6050 1000
 $Comp
-L Device:CP C65
+L Device:C_Polarized C65
 U 1 1 5E69E767
 P 6200 1800
+AR Path="/5E69E767" Ref="C65"  Part="1"
+AR Path="/5E8458FD/5E69E767" Ref="C65"  Part="1"
 F 0 "C65" V 5945 1800 50  0000 C CNN
 F 1 "220u" V 6036 1800 50  0000 C CNN
@@
 	6200 3700 6550 3700
 $Comp
-L Device:CP C63
+L Device:C_Polarized C63
 U 1 1 5E77E5F1
 P 6650 2600
+AR Path="/5E77E5F1" Ref="C63"  Part="1"
+AR Path="/5E8458FD/5E77E5F1" Ref="C63"  Part="1"
 F 0 "C63" H 6768 2646 50  0000 L CNN
 F 1 "1000u/16V" H 6768 2555 50  0000 L CNN
@@
 	6650 2850 6650 2750
 $Comp
-L Device:CP C66
+L Device:C_Polarized C66
 U 1 1 5E785362
 P 7950 1450
+AR Path="/5E785362" Ref="C66"  Part="1"
+AR Path="/5E8458FD/5E785362" Ref="C66"  Part="1"
 F 0 "C66" H 8068 1496 50  0000 L CNN
 F 1 "330u/35V" H 8068 1405 50  0000 L CNN
