File: 250469-RevA/user_port.sch (KiCad schematic (older format))
At the start: 16 parts, among them J2 Conn_02x12_Edge, U2 6526A, U22 7416, U23 74LS14

Commit message: Update schematic after changes in libs
Parts:
- C43: symbol Device:CP -> Device:C_Polarized
Changed lines of the file:
@@
 $EndComp
 $Comp
-L Device:CP C43
+L Device:C_Polarized C43
 U 1 1 5E332D3A
 P 4650 6650
+AR Path="/5E332D3A" Ref="C43"  Part="1"
+AR Path="/5E852F1D/5E332D3A" Ref="C43"  Part="1"
 F 0 "C43" H 4768 6696 50  0000 L CNN
 F 1 "220u" H 4768 6605 50  0000 L CNN
