File: 250469-RevA/video.sch (KiCad schematic (older format))
At the start: 19 parts, among them J5 DIN-8, M1 RF_Modulator, U20 8701, U21 4066, U7 8565, Y1 Crystal

Commit message: Updates and BOMs
Parts:
- CT1: footprint Capacitor_THT:C_Rect_L7.0mm_W6.5mm_P5.00mm -> Capacitor_SMD:C_Trimmer_Voltronics_JZ
Changed lines of the file:
@@
 F 0 "CT1" H 6716 5346 50  0000 L CNN
 F 1 "7.7-40p" H 6716 5255 50  0000 L CNN
-F 2 "Capacitor_THT:C_Rect_L7.0mm_W6.5mm_P5.00mm" H 6600 5300 50  0001 C CNN
+F 2 "Capacitor_SMD:C_Trimmer_Voltronics_JZ" H 6600 5300 50  0001 C CNN
 F 3 "~" H 6600 5300 50  0001 C CNN
 	1    6600 5300

Commit message: Add initial PCB with placed components
Parts:
- removed U7: 8565, Package_DIP:DIP-40_W15.24mm_Socket, symbol krl_MOS-Technology:8565
- added U7: 8565R2, Package_DIP:DIP-40_W15.24mm_Socket, symbol krl_MOS-Technology:8565R2
Connections:
- net +5V: now also U7.13 (VDD), U7.40 (VCC)
- net A10: now also U7.34 (A10)
- net A11: now also U7.23 (A11)
- net A8: now also U7.32 (A8)
- net A9: now also U7.33 (A9)
- net AEC: now also U7.16 (AEC)
- net BA: now also U7.12 (BA)
- net BTNA_LP: now also U7.9 (LP)
- net COLCLK: now also U7.21 (PHI_COL)
- net COLOR: now also U7.14 (COLOR)
- net D0: now also U7.7 (D0)
- net D1: now also U7.6 (D1)
- net D10: now also U7.36 (D10)
- net D11: now also U7.35 (D11)
- net D2: now also U7.5 (D2)
- net D3: now also U7.4 (D3)
- net D4: now also U7.3 (D4)
- net D5: now also U7.2 (D5)
- net D6: now also U7.1 (D6)
- net D7: now also U7.39 (D7)
- net D8: now also U7.38 (D8)
- net D9: now also U7.37 (D9)
- net DOTCLK: now also U7.22 (PHI_IN)
- net GND: now also U7.20 (GND)
- net MA0: now also U7.24 (A0/A8)
- net MA1: now also U7.25 (A1/A9)
- net MA2: now also U7.26 (A2/A10)
- net MA3: now also U7.27 (A3/A11)
- net MA4: now also U7.28 (A4/A12)
- net MA5: now also U7.29 (A5/A13)
- net PHI0: now also U7.17 (PHI0)
- net R~W: now also U7.11 (R/~W)
- net SL: now also U7.15 (SYNC/LUM)
- net VA6: now also U7.30 (A6)
- net VA7: now also U7.31 (A7)
- net ~IRQ: now also U7.8 (~IRQ)
- net ~RAS: now also U7.18 (~RAS)
- net ~VIC: now also U7.10 (~CS)
- net at JP4.2 (B): now also U7.19 (~CAS)
- net at L2.2: now also M1.1 (VCC)
- no-connect marks 3 -> 2
Other:
- note removed: "The RF Out goes to the antenna\nconnector integrated in the modulator"
Changed lines of the file:
@@
 $EndDescr
-$Comp
-L krl_MOS-Technology:8565 U7
-U 1 1 5E42887D
-P 2950 2750
-F 0 "U7" H 2600 3900 50  0000 C CNN
-F 1 "8565" H 3275 3900 50  0000 C CNN
-F 2 "Package_DIP:DIP-40_W15.24mm_Socket" H 2250 1550 50  0001 C CIN
-F 3 "" H 1750 3350 50  0001 C CNN
-	1    2950 2750
-	1    0    0    -1
-$EndComp
 $Comp
 L power:+5V #PWR0178
@@
 	5600 1150 5600 1250
 Wire Wire Line
-	6600 1150 7250 1150
-Wire Wire Line
-	7250 1150 7250 1600
+	6600 1150 7050 1150
+Wire Wire Line
+	7050 1150 7050 1600
 $Comp
 L power:GND #PWR0191
@@
 Wire Wire Line
 	5600 1600 5600 1550
-Text Notes 8150 1250 0    40   ~ 0
-The RF Out goes to the antenna\nconnector integrated in the modulator
-Wire Wire Line
-	8100 1900 8100 1350
-Wire Wire Line
-	8100 1350 8250 1350
-Wire Wire Line
-	7950 1900 8100 1900
-NoConn ~ 8250 1350
 Text GLabel 10200 2200 2    50   Input ~ 0
 AUDIO_OUT
@@
 L power:PWR_FLAG #FLG0101
 U 1 1 5E7E21E3
-P 7250 1150
-F 0 "#FLG0101" H 7250 1225 50  0001 C CNN
-F 1 "PWR_FLAG" H 7250 1323 50  0000 C CNN
-F 2 "" H 7250 1150 50  0001 C CNN
-F 3 "~" H 7250 1150 50  0001 C CNN
-	1    7250 1150
-	1    0    0    -1
-$EndComp
-Connection ~ 7250 1150
+P 7050 1075
+F 0 "#FLG0101" H 7050 1150 50  0001 C CNN
+F 1 "PWR_FLAG" H 7050 1248 50  0000 C CNN
+F 2 "" H 7050 1075 50  0001 C CNN
+F 3 "~" H 7050 1075 50  0001 C CNN
+	1    7050 1075
+	1    0    0    -1
+$EndComp
+Connection ~ 7050 1150
 Text Label 6000 2300 0    50   ~ 0
 AUDIO_OUT
@@
 Wire Wire Line
 	8350 5150 8500 5150
+$Comp
+L krl_MOS-Technology:8565R2 U7
+U 1 1 5EA66DAD
+P 2950 2750
+F 0 "U7" H 2600 3900 50  0000 C CNN
+F 1 "8565R2" H 3350 3900 50  0000 C CNN
+F 2 "Package_DIP:DIP-40_W15.24mm_Socket" H 2200 1500 50  0001 C CIN
+F 3 "" H 1800 3500 50  0001 C CNN
+	1    2950 2750
+	1    0    0    -1
+$EndComp
+Wire Wire Line
+	7050 1150 7050 1075
 Wire Bus Line
 	1950 2200 1950 2350

Commit message: Various improvements and changes to footprints
Parts:
- removed JP4: SolderJumper_2_Bridged, Jumper:SolderJumper-2_P1.3mm_Bridged_RoundedPad1.0x1.5mm, symbol Jumper:SolderJumper_2_Bridged
- CT1: footprint Capacitor_SMD:C_Trimmer_Voltronics_JZ -> krl_Capacitor_THT:C_Trimmer_JML_JML06_P5mm
- JP3: footprint Jumper:SolderJumper-2_P1.3mm_Bridged_RoundedPad1.0x1.5mm -> Connector_PinHeader_2.54mm:PinHeader_1x02_P2.54mm_Vertical
Connections:
- net ~CAS: now also U7.19 (~CAS)
Changed lines of the file:
@@
 Date "2020-04-15"
 Rev "1"
-Comp "https://github.com/orgs/KicadRetroArchive"
+Comp "https://github.com/KicadRetroArchive"
 Comment1 "KiCad schematic licensed under CERN-OHL-S"
 Comment2 "WARNING: These schematics might contain errors!"
@@
 F 0 "CT1" H 6716 5346 50  0000 L CNN
 F 1 "7.7-40p" H 6716 5255 50  0000 L CNN
-F 2 "Capacitor_SMD:C_Trimmer_Voltronics_JZ" H 6600 5300 50  0001 C CNN
+F 2 "krl_Capacitor_THT:C_Trimmer_JML_JML06_P5mm" H 6600 5300 50  0001 C CNN
 F 3 "~" H 6600 5300 50  0001 C CNN
 	1    6600 5300
@@
 F 0 "JP3" H 8850 5114 50  0000 C CNN
 F 1 "Jumper" H 8850 5023 50  0000 C CNN
-F 2 "Jumper:SolderJumper-2_P1.3mm_Bridged_RoundedPad1.0x1.5mm" H 8850 4850 50  0001 C CNN
+F 2 "Connector_PinHeader_2.54mm:PinHeader_1x02_P2.54mm_Vertical" H 8850 4850 50  0001 C CNN
 F 3 "~" H 8850 4850 50  0001 C CNN
 	1    8850 4850
@@
 Text Label 2050 2450 0    50   ~ 0
 VA7
-$Comp
-L Jumper:SolderJumper_2_Bridged JP4
-U 1 1 5E72030B
-P 2050 4150
-F 0 "JP4" H 2050 4050 50  0000 C CNN
-F 1 "SolderJumper_2_Bridged" H 2050 4264 50  0001 C CNN
-F 2 "Jumper:SolderJumper-2_P1.3mm_Bridged_RoundedPad1.0x1.5mm" H 2050 4150 50  0001 C CNN
-F 3 "~" H 2050 4150 50  0001 C CNN
-	1    2050 4150
-	1    0    0    -1
-$EndComp
-Wire Wire Line
-	2200 4150 2350 4150
-Wire Wire Line
-	1900 4150 1750 4150
+Wire Wire Line
+	1750 4150 2350 4150
 Wire Wire Line
 	3450 3550 3650 3550

Commit message: Changed footprint of DIC connectors and wiring of Color RAM
Parts:
- J5: footprint krl_Connector_DIN:CUI-Devices_SDS-80J_DIN-8_Circular -> krl_Connector_DIN:C64_Original_DIN-8_Circular
Changed lines of the file:
@@
 F 0 "J5" H 9150 1900 50  0000 C CNN
 F 1 "DIN-8" H 9600 1900 50  0000 C CNN
-F 2 "krl_Connector_DIN:CUI-Devices_SDS-80J_DIN-8_Circular" H 9350 2200 50  0001 C CNN
+F 2 "krl_Connector_DIN:C64_Original_DIN-8_Circular" H 9350 2200 50  0001 C CNN
 F 3 "http://www.mouser.com/ds/2/18/40_c091_abd_e-75918.pdf" H 9350 2200 50  0001 C CNN
 	1    9350 2200

Commit message: Update schematic after changes in libs
Parts:
- C36: symbol Device:CP -> Device:C_Polarized
- CT1: symbol Device:CTRIM -> Device:C_Trim
- FB1: symbol Device:Ferrite_Bead -> Device:FerriteBead
- FB2, FB3, FB4: symbol Device:Ferrite_Bead_Small -> Device:FerriteBead_Small
- JP3: symbol Device:Jumper -> Jumper:Jumper_2_Bridged
Other:
- moved on the sheet: Y1
Changed lines of the file:
@@
 $EndComp
 $Comp
-L Device:CP C36
+L Device:C_Polarized C36
 U 1 1 5E431A66
 P 1900 5200
+AR Path="/5E431A66" Ref="C36"  Part="1"
+AR Path="/5E427C5E/5E431A66" Ref="C36"  Part="1"
 F 0 "C36" H 2018 5246 50  0000 L CNN
 F 1 "47u/16V" H 2018 5155 50  0000 L CNN
@@
 L Device:Crystal Y1
 U 1 1 5E494D12
-P 6600 4725
-F 0 "Y1" V 6600 4875 50  0000 L CNN
-F 1 "Crystal" V 6645 4856 50  0001 L CNN
-F 2 "Crystal:Crystal_HC49-U_Vertical" H 6600 4725 50  0001 C CNN
-F 3 "~" H 6600 4725 50  0001 C CNN
-	1    6600 4725
+P 6600 4700
+F 0 "Y1" V 6600 4850 50  0000 L CNN
+F 1 "Crystal" V 6645 4831 50  0001 L CNN
+F 2 "Crystal:Crystal_HC49-U_Vertical" H 6600 4700 50  0001 C CNN
+F 3 "~" H 6600 4700 50  0001 C CNN
+	1    6600 4700
 	0    -1   1    0
 $EndComp
@@
 	6850 4500 6600 4500
 Wire Wire Line
-	6600 4500 6600 4575
-Wire Wire Line
 	7150 4950 6600 4950
 $Comp
-L Device:CTRIM CT1
+L Device:C_Trim CT1
 U 1 1 5E49D621
 P 6600 5300
+AR Path="/5E49D621" Ref="CT1"  Part="1"
+AR Path="/5E427C5E/5E49D621" Ref="CT1"  Part="1"
 F 0 "CT1" H 6716 5346 50  0000 L CNN
 F 1 "7.7-40p" H 6716 5255 50  0000 L CNN
@@
 Wire Wire Line
 	6600 4950 6600 5150
-Connection ~ 6600 4950
 Wire Wire Line
 	6600 5450 6600 5600
@@
 NoConn ~ 6950 5150
 $Comp
-L Device:Jumper JP3
+L Jumper:Jumper_2_Bridged JP3
 U 1 1 5E4A291C
 P 8850 4850
-F 0 "JP3" H 8850 5114 50  0000 C CNN
-F 1 "Jumper" H 8850 5023 50  0000 C CNN
+AR Path="/5E4A291C" Ref="JP3"  Part="1"
+AR Path="/5E427C5E/5E4A291C" Ref="JP3"  Part="1"
+F 0 "JP3" H 8850 5100 50  0000 C CNN
+F 1 "Jumper" H 8850 5000 50  0000 C CNN
 F 2 "Connector_PinHeader_2.54mm:PinHeader_1x02_P2.54mm_Vertical" H 8850 4850 50  0001 C CNN
 F 3 "~" H 8850 4850 50  0001 C CNN
@@
 	-1   0    0    -1
 $EndComp
-Wire Wire Line
-	8550 4850 8350 4850
-Wire Wire Line
-	9150 4850 9250 4850
 Wire Wire Line
 	9250 4850 9250 4950
@@
 $EndComp
 $Comp
-L Device:Ferrite_Bead FB1
+L Device:FerriteBead FB1
 U 1 1 5E4A5ABB
 P 8950 5550
+AR Path="/5E4A5ABB" Ref="FB1"  Part="1"
+AR Path="/5E427C5E/5E4A5ABB" Ref="FB1"  Part="1"
 F 0 "FB1" V 8750 5550 50  0000 C CNN
 F 1 "2 Turns" V 9133 5550 50  0000 C CNN
@@
 	8750 2200 9050 2200
 $Comp
-L Device:Ferrite_Bead_Small FB4
+L Device:FerriteBead_Small FB4
 U 1 1 5E508AB5
 P 8650 1850
+AR Path="/5E508AB5" Ref="FB4"  Part="1"
+AR Path="/5E427C5E/5E508AB5" Ref="FB4"  Part="1"
 F 0 "FB4" V 8505 1850 50  0000 C CNN
 F 1 "Ferrite_Bead_Small" V 8504 1850 50  0001 C CNN
@@
 $EndComp
 $Comp
-L Device:Ferrite_Bead_Small FB3
+L Device:FerriteBead_Small FB3
 U 1 1 5E5084E2
 P 8650 2200
+AR Path="/5E5084E2" Ref="FB3"  Part="1"
+AR Path="/5E427C5E/5E5084E2" Ref="FB3"  Part="1"
 F 0 "FB3" V 8505 2200 50  0000 C CNN
 F 1 "Ferrite_Bead_Small" V 8504 2200 50  0001 C CNN
@@
 $EndComp
 $Comp
-L Device:Ferrite_Bead_Small FB2
+L Device:FerriteBead_Small FB2
 U 1 1 5E507BD4
 P 8650 2550
+AR Path="/5E507BD4" Ref="FB2"  Part="1"
+AR Path="/5E427C5E/5E507BD4" Ref="FB2"  Part="1"
 F 0 "FB2" V 8505 2550 50  0000 C CNN
 F 1 "Ferrite_Bead_Small" V 8504 2550 50  0001 C CNN
@@
 Wire Wire Line
 	2050 3450 2450 3450
-Connection ~ 6600 4575
-Wire Wire Line
-	6600 4575 6600 4650
-Wire Wire Line
-	6600 4875 6600 4950
 Wire Wire Line
 	6950 5150 7150 5150
@@
 Wire Wire Line
 	7050 1150 7050 1075
+Wire Wire Line
+	6600 4550 6600 4500
+Wire Wire Line
+	6600 4850 6600 4950
+Connection ~ 6600 4950
+Wire Wire Line
+	9050 4850 9250 4850
+Wire Wire Line
+	8350 4850 8650 4850
 Wire Bus Line
 	1950 2200 1950 2350
