File: 250469-RevA/joystick.kicad_sch (KiCad schematic)
At the start: 17 parts, among them J11 DE9_Plug, J9 DE9_Plug, U18 4066

Commit message: Footprints and Symbols updates
Parts:
- J11, J9: footprint (none) -> 250469-01:DSUB-9_Male_Joystick
Changed lines of the file:
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@@
       (effects (font (size 1.27 1.27)))
     )
-    (property "Footprint" "" (at 180.34 114.3 0)
+    (property "Footprint" "250469-01:DSUB-9_Male_Joystick" (at 180.34 114.3 0)
       (effects (font (size 1.27 1.27)) hide)
     )
@@
       (effects (font (size 1.27 1.27)) (justify left))
     )
-    (property "Footprint" "" (at 148.59 64.77 0)
+    (property "Footprint" "250469-01:DSUB-9_Male_Joystick" (at 148.59 64.77 0)
       (effects (font (size 1.27 1.27)) hide)
     )

Commit message: Fixes after renaming the project library
Parts:
- J11, J9: footprint 250469-01:DSUB-9_Male_Joystick -> C64-C-250469:DSUB-9_Male_Joystick
- L3: footprint 250469-01:L_Radial_L7.5mm_W3mm_P5.00mm_Kemet_SBT-02 -> C64-C-250469:L_Radial_L7.5mm_W3mm_P5.00mm_Kemet_SBT-02
Changed lines of the file:
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@@
       (effects (font (size 1.27 1.27)))
     )
-    (property "Footprint" "250469-01:L_Radial_L7.5mm_W3mm_P5.00mm_Kemet_SBT-02" (at 240.03 147.32 0)
+    (property "Footprint" "C64-C-250469:L_Radial_L7.5mm_W3mm_P5.00mm_Kemet_SBT-02" (at 240.03 147.32 0)
       (effects (font (size 1.27 1.27)) hide)
     )
@@
       (effects (font (size 1.27 1.27)))
     )
-    (property "Footprint" "250469-01:DSUB-9_Male_Joystick" (at 180.34 114.3 0)
+    (property "Footprint" "C64-C-250469:DSUB-9_Male_Joystick" (at 180.34 114.3 0)
       (effects (font (size 1.27 1.27)) hide)
     )
@@
       (effects (font (size 1.27 1.27)) (justify left))
     )
-    (property "Footprint" "250469-01:DSUB-9_Male_Joystick" (at 148.59 64.77 0)
-      (effects (font (size 1.27 1.27)) hide)
-    )
+    (property "Footprint" "C64-C-250469:DSUB-9_Male_Joystick" (at 148.59 64.77 0)
+      (effects (font (size 1.27 1.27)) hide)
+    )
